File: project/BreakoutBoard_2.brd (EAGLE design)
At the start: 45.2 x 45.2 mm, 2 parts, among them J1 XF2L-2435-1, X1 LCD

Commit message: WIP
Parts:
- moved J1 9.22 mm to (16.0, 16.0), flipped to the top
Routing:
- net N$19: track 30.5 -> 0.00 mm, vias 1 -> 0
- net N$20: track 30.1 -> 0.00 mm, vias 1 -> 0
- net N$21: track 29.6 -> 0.00 mm, vias 1 -> 0
- net N$22: track 29.2 -> 0.00 mm, vias 1 -> 0
- net N$23: track 28.4 -> 0.00 mm, vias 1 -> 0
- net N$24: track 27.3 -> 0.00 mm, vias 1 -> 0
- net N$13: track 29.1 -> 14.5 mm, vias 1 -> 0
- net N$14: track 29.6 -> 16.1 mm, vias 1 -> 0
- net N$15: track 30.0 -> 17.6 mm, vias 1 -> 0
- net N$1: track 21.1 -> 8.77 mm, vias 1 -> 0
- net N$2: track 20.7 -> 8.73 mm, vias 1 -> 0
- net N$3: track 20.3 -> 8.69 mm, vias 1 -> 0
- net N$4: track 20.0 -> 8.65 mm, vias 1 -> 0
- net N$16: track 30.4 -> 19.1 mm, vias 1 -> 0
- net N$5: track 19.6 -> 8.60 mm, vias 1 -> 0
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